File: pcb/aquaponics-1.kicad_pcb (KiCad board)
At the start: 2 copper layers, 52.1 x 63.5 mm, 19 parts, among them J1 5V Power Source, J2 Screw_Terminal_01x02, J3 Water Level Sensor, J4 Rain Sensor, J5 Conn_01x02_Female, M1 Growbed Pump, M2 Overflow Pump, M3 Fish Feeder, Q1 TIP120, Q2 TIP120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

Commit message: Update PCB /
Parts:
- added D1: DIODE, Diode_THT:D_DO-15_P2.54mm_Vertical_AnodeUp, F.Cu at (39.4, 19.1)
- R3: value 330 -> 10k
- moved J1 3.17 mm to (50.2, 71.1)
- moved J5 3.17 mm to (65.4, 71.3)
Connections:
- J2 pad 2: GND -> Net-(D1-Pad1)
- U1 pad 16: Net-(U1-Pad16) -> Net-(R6-Pad1)
- U1 pad 19: Net-(R6-Pad1) -> Net-(U1-Pad19)
Routing:
- net Net-(J2-Pad1): track 95.6 -> 53.6 mm
- net Net-(D1-Pad1): track 0.00 -> 17.8 mm
- net GND: track 131.9 -> 126.0 mm
- net Net-(R6-Pad1): track 23.3 -> 27.6 mm
- net +5V: track 68.1 -> 71.3 mm
- net Net-(M2-Pad2): track 7.89 -> 4.81 mm
- net Net-(M1-Pad2): track 7.25 -> 4.81 mm
- net Net-(M3-Pad2): track 6.35 -> 4.81 mm
