File: pcb/aquaponics-1.kicad_pcb (KiCad board)
At the start: 2 copper layers, 54 x 63.5 mm, 20 parts, among them J1 5V Power Source, J2 Screw_Terminal_01x02, J3 Water Level Sensor, J4 Rain Sensor, J5 Conn_01x02_Female, M1 Growbed Pump, M2 Overflow Pump, M3 Fish Feeder, Q1 TIP120, Q2 TIP120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

Commit message: Version 2 board
Parts:
- added J6: Conn_01x04_Female, Connector_PinHeader_2.54mm:PinHeader_1x04_P2.54mm_Vertical, F.Cu at (39.4, 73.7)
Routing:
- net Net-(J6-Pad1): track 0.00 -> 29.6 mm
- net Net-(J6-Pad2): track 0.00 -> 26.0 mm
- net GND1: track 71.6 -> 83.9 mm
- net +5V: track 67.4 -> 79.1 mm

Commit message: Update PCB model
Routing:
- net +5V: track 79.1 -> 73.9 mm

Commit message: Temp sensor to use 5V souce
Connections:
- R6 pad 2: +3V3 -> +5V
- U1 pad 17: +3V3 -> Net-(U1-Pad17)
- U2 pad 1: +3V3 -> +5V
Routing:
- net +5V: track 73.9 -> 99.0 mm
- net +3V3: track 18.3 -> 0.00 mm
